File: Hardware/PCB/Hornbill Lights/Hornbill Lights.kicad_pcb (KiCad board)
At the start: 2 copper layers, 93 x 60 mm, 57 parts, among them CON1 USB-MINI-B, CON2 BARREL_JACK, M1 ESP-WROOM-32, P1 CONN_01X14, P10 CONN_01X14, P11 CONN_01X14, P12 CONN_01X14, P13 CONN_01X14, P14 CONN_01X14, P15 CONN_01X14, P2 CONN_01X03, P3 CONN_01X14, P4 CONN_01X14, P5 CONN_01X14, P6 CONN_01X14, P7 CONN_01X14, P8 CONN_01X14, P9 CONN_01X14, Q3 S8050, Q4 S8050, SW1 SW_PUSH, SW2 SW_PUSH, U1 AP2112K, U2 OSH_Symbol, U3 EE_Logo, U4 EE_Logo, U5 MountingHole, U6 MountingHole, U7 MountingHole, U8 MountingHole, U9 CP2102, Y1 32.768KHz RTC Crystal

Commit message: PCB Layout Updated
Parts:
- removed P10, P11, P12, P13, P14, P15, P3, P4, P5, P6, P7, P8, P9: CONN_01X14, Explore:EE_Pin_Header_Straight_1x14_Pitch2.54mm
- added D1: D, Explore:SOD-80_diode_1, F.Cu at (141.7, 84.8)
- C9, CON2, U2, U4: moved to B.Cu
- P1: value CONN_01X14 -> CONN_01X03; footprint Explore:EE_Pin_Header_Straight_1x14_Pitch2.54mm -> Pin_Headers:Pin_Header_Straight_1x03_Pitch2.54mm
- P2: footprint Pin_Headers:Pin_Header_Angled_1x03_Pitch2.54mm -> Pin_Headers:Pin_Header_Straight_1x03_Pitch2.54mm
- moved P1 66.8 mm to (81.3, 85.1), turned to 180 degrees
- moved U4 48.4 mm to (145.2, 97.5), turned to 180 degrees
- moved C7 45.4 mm to (142.5, 96.3), turned to 270 degrees
- moved R5 44.9 mm to (129.8, 80.0)
- moved U2 44.4 mm to (131.6, 121.8), turned to 180 degrees
- moved C1 40.4 mm to (101.6, 77.7), turned to 90 degrees
- moved R11 38.7 mm to (129.8, 82.3)
- moved R12 37.2 mm to (129.8, 85.9), turned to 270 degrees
- moved C2 35.9 mm to (104.6, 77.7), turned to 90 degrees
- moved C4 33.2 mm to (102.4, 83.1), turned to 180 degrees
- moved D2 31.6 mm to (97.5, 93.5)
- moved SW1 31.1 mm to (101.1, 70.1)
- moved R2 30.7 mm to (96.9, 70.1)
- moved C5 30.0 mm to (102.4, 90.2), turned to 180 degrees
- moved Y1 29.3 mm to (103.1, 86.6), turned to 270 degrees
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Connections:
- C7 pad 2: +5V -> VCC
- F1 pad 1: +5V -> VCC
- P1 pad 1: Net-(P1-Pad1) -> +5V
- P1 pad 3: Net-(P1-Pad3) -> GND
- P2 pad 2: Net-(P2-Pad2) -> Net-(P1-Pad2)
- R12 pad 1: Net-(P2-Pad2) -> Net-(P1-Pad2)
- U9 pad 7: +5V -> VCC
- U9 pad 8: +5V -> VCC
Routing:
- net GND: track 0.00 -> 271.3 mm, vias 0 -> 11
- net +5V: track 0.00 -> 155.2 mm, vias 0 -> 4
- net +3V3: track 0.00 -> 92.3 mm, vias 0 -> 4
- net /EN: track 0.00 -> 81.1 mm, vias 0 -> 6
- net /IO0: track 0.00 -> 69.1 mm, vias 0 -> 2
- net Net-(P1-Pad2): track 0.00 -> 66.4 mm, vias 0 -> 1
- net /RTS: track 0.00 -> 47.5 mm
- net Net-(R11-Pad2): track 0.00 -> 37.6 mm, vias 0 -> 2
- net Net-(R5-Pad2): track 0.00 -> 36.2 mm, vias 0 -> 2
- net VCC: track 0.00 -> 33.0 mm, vias 0 -> 2
- net Net-(R3-Pad2): track 0.00 -> 23.2 mm
- net /DTR: track 0.00 -> 23.0 mm, vias 0 -> 2
- net /IO13: track 0.00 -> 15.5 mm
- net Net-(CON1-Pad3): track 0.00 -> 14.3 mm, vias 0 -> 2
- net Net-(CON1-Pad2): track 0.00 -> 10.9 mm
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Other:
- net class Default: clearance 0.2 -> 0.15
- rule trace_clearance: 0.2 -> 0.15
- board text added: "Exploreembedded.com"

Commit message: Added protype pads
Parts:
- added P10: CONN_01X11, Explore:Pin_Header_Straight_1x11_Pitch2.54mm, F.Cu at (96.5, 121.9)
- added P11: CONN_01X11, Explore:Pin_Header_Straight_1x11_Pitch2.54mm, F.Cu at (96.5, 124.5)
- added P3: CONN_01X11, Explore:Pin_Header_Straight_1x11_Pitch2.54mm, F.Cu at (96.5, 104.1)
- added P4: CONN_01X11, Explore:Pin_Header_Straight_1x11_Pitch2.54mm, F.Cu at (96.5, 106.7)
- added P5: CONN_01X11, Explore:Pin_Header_Straight_1x11_Pitch2.54mm, F.Cu at (96.5, 109.2)
- added P6: CONN_01X11, Explore:Pin_Header_Straight_1x11_Pitch2.54mm, F.Cu at (96.5, 111.8)
- added P7: CONN_01X11, Explore:Pin_Header_Straight_1x11_Pitch2.54mm, F.Cu at (96.5, 114.3)
- added P8: CONN_01X11, Explore:Pin_Header_Straight_1x11_Pitch2.54mm, F.Cu at (96.5, 116.8)
- added P9: CONN_01X11, Explore:Pin_Header_Straight_1x11_Pitch2.54mm, F.Cu at (96.5, 119.4)
- moved D2 31.7 mm to (128.3, 101.2), turned to 180 degrees
- moved R6 27.7 mm to (128.3, 98.8)
- moved R7 25.2 mm to (129.0, 95.8), turned to 270 degrees
- moved U2 16.6 mm to (148.2, 122.0)
- moved C9 5.69 mm to (90.4, 104.5), turned to 180 degrees
- moved U3 5.36 mm to (139.8, 118.1)
Connections:
- M1 pad 29: Net-(M1-Pad29) -> /IO5
- R7 pad 1: /IO13 -> /IO5
Routing:
- net GND: track 271.3 -> 300.6 mm, vias 11 -> 12
- net /IO5: track 0.00 -> 13.6 mm, vias 0 -> 2
- net /IO13: track 15.5 -> 6.56 mm
- net +5V: track 155.2 -> 152.6 mm
Other:
- board text added: "DATA"
- board text added: "GND"
- board text added: "VCC"
