File: Hardware/PCB/Hornbill Lights/Hornbill Lights.kicad_pcb (KiCad board)
At the start: 2 copper layers, 93 x 60 mm, 54 parts, among them CON1 USB-MINI-B, CON2 BARREL_JACK, M1 ESP-WROOM-32, P1 CONN_01X03, P10 CONN_01X11, P11 CONN_01X11, P2 CONN_01X03, P3 CONN_01X11, P4 CONN_01X11, P5 CONN_01X11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

Commit message: Gerber data generated for v0.1
Other:
- board text added: "v0.1"
