File: Hardware/PCB/Hornbill Lights/Hornbill Lights.sch (KiCad schematic (older format))
At the start: 57 parts, among them CON1 USB-MINI-B, CON2 BARREL_JACK, M1 ESP-WROOM-32, P1 CONN_01X14, P10 CONN_01X14, P11 CONN_01X14, P12 CONN_01X14, P13 CONN_01X14, P14 CONN_01X14, P15 CONN_01X14, P2 CONN_01X03, P3 CONN_01X14, P4 CONN_01X14, P5 CONN_01X14, P6 CONN_01X14, P7 CONN_01X14, P8 CONN_01X14, P9 CONN_01X14, Q3 S8050, Q4 S8050, SW1 SW_PUSH, SW2 SW_PUSH, U1 AP2112K, U2 OSH_Symbol, U3 EE_Logo, U4 EE_Logo, U5 MountingHole, U6 MountingHole, U7 MountingHole, U8 MountingHole, U9 CP2102, Y1 32.768KHz RTC Crystal

Commit message: PCB Layout Updated
Parts:
- removed P1, P10, P11, P12, P13, P14, P15, P3, P4, P5, P6, P7, P8, P9: CONN_01X14, Explore:EE_Pin_Header_Straight_1x14_Pitch2.54mm, symbol CONN_01X14
- added D1: D, Explore:SOD-80_diode_1, symbol D
- added P1: CONN_01X03, Pin_Headers:Pin_Header_Straight_1x03_Pitch2.54mm, symbol CONN_01X03
- P2: footprint Pin_Headers:Pin_Header_Angled_1x03_Pitch2.54mm -> Pin_Headers:Pin_Header_Straight_1x03_Pitch2.54mm
Connections:
- net +5V: now also D1.1 (K), P1.1 (P1); no longer C7.2, F1.1, U9.7 (REGIN), U9.8 (VBUS)
- net GND: now also P1.3 (P3)
- net at P2.2 (P2), R12.1: now also P1.2 (P2)
- new net VCC: C7.2, D1.2 (A), F1.1, U9.7 (REGIN), U9.8 (VBUS)
- no-connect marks 243 -> 47

Commit message: Added protype pads
Parts:
- added P10, P11, P3, P4, P5, P6, P7, P8, P9: CONN_01X11, Explore:Pin_Header_Straight_1x11_Pitch2.54mm, symbol CONN_01X11
Connections:
- net IO13: no longer R7.1
- net IO5: now reaches M1.29 (IO5)
- net IO5: now also R7.1
- no-connect marks 47 -> 145
Changed lines of the file:
@@
 Text Label 4800 5110 0    60   ~ 0
 TXD0
-Text Label 3450 6410 3    60   ~ 0
-IO13
 Text Label 4150 6410 3    60   ~ 0
 IO15
@@
 NoConn ~ 4800 5510
 NoConn ~ 4800 5610
-NoConn ~ 4800 5710
 NoConn ~ 4800 6010
 NoConn ~ 4250 6410
@@
 	3150 6620 3150 6630
 Wire Wire Line
-	3450 6410 3450 6980
-Wire Wire Line
 	2040 1525 1920 1525
 Wire Wire Line
@@
 Wire Wire Line
 	1050 1265 1050 1375
+Text Label 4800 5710 0    60   ~ 0
+IO5
+Text Label 3450 6980 0    60   ~ 0
+IO5
+Text Label 3450 6410 3    60   ~ 0
+IO13
+$Comp
+L CONN_01X11 P3
+U 1 1 59245B5B
+P 12300 1800
+F 0 "P3" H 12300 2400 50  0000 C CNN
+F 1 "CONN_01X11" V 12400 1800 50  0000 C CNN
+F 2 "Explore:Pin_Header_Straight_1x11_Pitch2.54mm" H 12300 1800 50  0001 C CNN
+F 3 "" H 12300 1800 50  0000 C CNN
+	1    12300 1800
+	1    0    0    -1
+$EndComp
+$Comp
+L CONN_01X11 P5
+U 1 1 59245C0C
+P 12700 1800
+F 0 "P5" H 12700 2400 50  0000 C CNN
+F 1 "CONN_01X11" V 12800 1800 50  0000 C CNN
+F 2 "Explore:Pin_Header_Straight_1x11_Pitch2.54mm" H 12700 1800 50  0001 C CNN
+F 3 "" H 12700 1800 50  0000 C CNN
+	1    12700 1800
+	1    0    0    -1
+$EndComp
+$Comp
+L CONN_01X11 P7
+U 1 1 59245CAD
+P 13100 1800
+F 0 "P7" H 13100 2400 50  0000 C CNN
+F 1 "CONN_01X11" V 13200 1800 50  0000 C CNN
+F 2 "Explore:Pin_Header_Straight_1x11_Pitch2.54mm" H 13100 1800 50  0001 C CNN
+F 3 "" H 13100 1800 50  0000 C CNN
+	1    13100 1800
+	1    0    0    -1
+$EndComp
+$Comp
+L CONN_01X11 P9
+U 1 1 59245D55
+P 13500 1800
+F 0 "P9" H 13500 2400 50  0000 C CNN
+F 1 "CONN_01X11" V 13600 1800 50  0000 C CNN
+F 2 "Explore:Pin_Header_Straight_1x11_Pitch2.54mm" H 13500 1800 50  0001 C CNN
+F 3 "" H 13500 1800 50  0000 C CNN
+	1    13500 1800
+	1    0    0    -1
+$EndComp
+$Comp
+L CONN_01X11 P11
+U 1 1 59245DFC
+P 13900 1800
+F 0 "P11" H 13900 2400 50  0000 C CNN
+F 1 "CONN_01X11" V 14000 1800 50  0000 C CNN
+F 2 "Explore:Pin_Header_Straight_1x11_Pitch2.54mm" H 13900 1800 50  0001 C CNN
+F 3 "" H 13900 1800 50  0000 C CNN
+	1    13900 1800
+	1    0    0    -1
+$EndComp
+$Comp
+L CONN_01X11 P4
+U 1 1 592460B0
+P 12300 3050
+F 0 "P4" H 12300 3650 50  0000 C CNN
+F 1 "CONN_01X11" V 12400 3050 50  0000 C CNN
+F 2 "Explore:Pin_Header_Straight_1x11_Pitch2.54mm" H 12300 3050 50  0001 C CNN
+F 3 "" H 12300 3050 50  0000 C CNN
+	1    12300 3050
+	1    0    0    -1
+$EndComp
+$Comp
+L CONN_01X11 P6
+U 1 1 59246169
+P 12700 3050
+F 0 "P6" H 12700 3650 50  0000 C CNN
+F 1 "CONN_01X11" V 12800 3050 50  0000 C CNN
+F 2 "Explore:Pin_Header_Straight_1x11_Pitch2.54mm" H 12700 3050 50  0001 C CNN
+F 3 "" H 12700 3050 50  0000 C CNN
+	1    12700 3050
+	1    0    0    -1
+$EndComp
+$Comp
+L CONN_01X11 P8
+U 1 1 59246229
+P 13100 3050
+F 0 "P8" H 13100 3650 50  0000 C CNN
+F 1 "CONN_01X11" V 13200 3050 50  0000 C CNN
+F 2 "Explore:Pin_Header_Straight_1x11_Pitch2.54mm" H 13100 3050 50  0001 C CNN
+F 3 "" H 13100 3050 50  0000 C CNN
+	1    13100 3050
+	1    0    0    -1
+$EndComp
+$Comp
+L CONN_01X11 P10
+U 1 1 592462E8
+P 13500 3050
+F 0 "P10" H 13500 3650 50  0000 C CNN
+F 1 "CONN_01X11" V 13600 3050 50  0000 C CNN
+F 2 "Explore:Pin_Header_Straight_1x11_Pitch2.54mm" H 13500 3050 50  0001 C CNN
+F 3 "" H 13500 3050 50  0000 C CNN
+	1    13500 3050
+	1    0    0    -1
+$EndComp
+NoConn ~ 12100 1300
+NoConn ~ 12100 1400
+NoConn ~ 12100 1500
+NoConn ~ 12100 1600
+NoConn ~ 12100 1700
+NoConn ~ 12100 1800
+NoConn ~ 12100 1900
+NoConn ~ 12100 2000
+NoConn ~ 12100 2100
+NoConn ~ 12100 2200
+NoConn ~ 12100 2300
+NoConn ~ 12500 1300
+NoConn ~ 12500 1400
+NoConn ~ 12500 1500
+NoConn ~ 12500 1600
+NoConn ~ 12500 1700
+NoConn ~ 12500 1800
+NoConn ~ 12500 1900
+NoConn ~ 12500 2000
+NoConn ~ 12500 2100
+NoConn ~ 12500 2200
+NoConn ~ 12500 2300
+NoConn ~ 12900 1300
+NoConn ~ 12900 1400
+NoConn ~ 12900 1500
+NoConn ~ 12900 1600
+NoConn ~ 12900 1700
+NoConn ~ 12900 1800
+NoConn ~ 12900 1900
+NoConn ~ 12900 2000
+NoConn ~ 12900 2100
+NoConn ~ 12900 2200
+NoConn ~ 12900 2300
+NoConn ~ 13300 1300
+NoConn ~ 13300 1400
+NoConn ~ 13300 1500
+NoConn ~ 13300 1600
+NoConn ~ 13300 1700
+NoConn ~ 13300 1800
+NoConn ~ 13300 1900
+NoConn ~ 13300 2000
+NoConn ~ 13300 2100
+NoConn ~ 13300 2200
+NoConn ~ 13300 2300
+NoConn ~ 13700 1300
+NoConn ~ 13700 1400
+NoConn ~ 13700 1500
+NoConn ~ 13700 1600
+NoConn ~ 13700 1700
+NoConn ~ 13700 1800
+NoConn ~ 13700 1900
+NoConn ~ 13700 2000
+NoConn ~ 13700 2100
+NoConn ~ 13700 2200
+NoConn ~ 13700 2300
+NoConn ~ 12100 2550
+NoConn ~ 12100 2650
+NoConn ~ 12100 2750
+NoConn ~ 12100 2850
+NoConn ~ 12100 2950
+NoConn ~ 12100 3050
+NoConn ~ 12100 3150
+NoConn ~ 12100 3250
+NoConn ~ 12100 3350
+NoConn ~ 12100 3450
+NoConn ~ 12100 3550
+NoConn ~ 12500 2550
+NoConn ~ 12500 2650
+NoConn ~ 12500 2750
+NoConn ~ 12500 2850
+NoConn ~ 12500 2950
+NoConn ~ 12500 3050
+NoConn ~ 12500 3150
+NoConn ~ 12500 3250
+NoConn ~ 12500 3350
+NoConn ~ 12500 3450
+NoConn ~ 12500 3550
+NoConn ~ 12900 2550
+NoConn ~ 12900 2650
+NoConn ~ 12900 2750
+NoConn ~ 12900 2850
+NoConn ~ 12900 2950
+NoConn ~ 12900 3050
+NoConn ~ 12900 3150
+NoConn ~ 12900 3250
+NoConn ~ 12900 3350
+NoConn ~ 12900 3450
+NoConn ~ 12900 3550
+NoConn ~ 13300 2550
+NoConn ~ 13300 2650
+NoConn ~ 13300 2750
+NoConn ~ 13300 2850
+NoConn ~ 13300 2950
+NoConn ~ 13300 3050
+NoConn ~ 13300 3150
+NoConn ~ 13300 3250
+NoConn ~ 13300 3350
+NoConn ~ 13300 3450
+NoConn ~ 13300 3550
 $EndSCHEMATC
